Commit message: various changes to make it work properly

File: panda_description/urdf/panda.urdf.xacro (robot description, xacro)
@@ -1,5 +1,5 @@
 <?xml version="1.0"?>
 <!-- URDF for Franka Emika Panda -->
-<robot xmlns:xacro="http://wiki.ros.org/xacro" name="$(arg name)">
+<robot xmlns:xacro="http://wiki.ros.org/xacro" name="panda">
   <!--                   -->
   <!-- Imported elements -->
@@ -61,7 +61,16 @@
     gazebo_preserve_fixed_joint="$(arg gazebo_preserve_fixed_joint)"
   />
+  <joint name="${world_name}_to_base_link" type="fixed">
+      <!-- <origin xyz="${world_xyz}" rpy="${world_rpy}"/> -->
+      <parent link="${world_name}"/>
+      <child link="base_link"/>
+  </joint>
+  <xacro:panda_dummy_link
+    link_name="base_link"
+    gazebo_preserve_fixed_joint="$(arg gazebo_preserve_fixed_joint)"
+  />
   <!-- Arm -->
   <xacro:panda_arm
-    base_parent="world"
+    base_parent="base_link"
     prefix="${prefix_arm}"
     origin_xyz="${origin_xyz}"

File: panda_description/urdf/panda_utils.xacro (robot description, xacro)
@@ -22,5 +22,5 @@
         <origin xyz="0 0 0" rpy="${mesh_offset_rpy}"/>
         <geometry>
-          <mesh filename="package://panda_description/meshes/visual/${mesh}.dae"/>
+          <mesh filename="package://panda_description/panda/meshes/visual/${mesh}.dae"/>
         </geometry>
       </visual>
@@ -29,5 +29,5 @@
           <origin xyz="0 0 0" rpy="${mesh_offset_rpy}"/>
           <geometry>
-            <mesh filename="package://panda_description/meshes/collision/${mesh}.stl"/>
+            <mesh filename="package://panda_description/panda/meshes/collision/${mesh}.stl"/>
           </geometry>
         </collision>
