Commit message: new branch

File: panda_description/urdf/panda.urdf (robot description, URDF)
Before this commit: robot panda, 14 links, 13 joints
Links:
- added link base_link
- link panda_hand: geometry collision mesh filename=package://panda_description/panda/meshes/collision/hand.stl; visual mesh filename=package://panda_description/panda/meshes/visual/hand.dae
- link panda_leftfinger: geometry collision mesh filename=package://panda_description/panda/meshes/collision/finger.s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; visual mesh filename=package://panda_description/panda/meshes/visual/finger.dae
- link panda_link0: geometry collision mesh filename=package://panda_description/panda/meshes/collision/link0.stl; visual mesh filename=package://panda_description/panda/meshes/visual/link0.dae
- link panda_link1: geometry collision mesh filename=package://panda_description/panda/meshes/collision/link1.stl; visual mesh filename=package://panda_description/panda/meshes/visual/link1.dae
- link panda_link2: geometry collision mesh filename=package://panda_description/panda/meshes/collision/link2.stl; visual mesh filename=package://panda_description/panda/meshes/visual/link2.dae
- link panda_link3: geometry collision mesh filename=package://panda_description/panda/meshes/collision/link3.stl; visual mesh filename=package://panda_description/panda/meshes/visual/link3.dae
- link panda_link4: geometry collision mesh filename=package://panda_description/panda/meshes/collision/link4.stl; visual mesh filename=package://panda_description/panda/meshes/visual/link4.dae
- link panda_link5: geometry collision mesh filename=package://panda_description/panda/meshes/collision/link5.stl; visual mesh filename=package://panda_description/panda/meshes/visual/link5.dae
- link panda_link6: geometry collision mesh filename=package://panda_description/panda/meshes/collision/link6.stl; visual mesh filename=package://panda_description/panda/meshes/visual/link6.dae
- link panda_link7: geometry collision mesh filename=package://panda_description/panda/meshes/collision/link7.stl; visual mesh filename=package://panda_description/panda/meshes/visual/link7.dae
- link panda_rightfinger: geometry collision mesh filename=package://panda_description/panda/meshes/collision/finger.s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; visual mesh filename=package://panda_description/panda/meshes/visual/finger.dae
Joints:
- added joint world_to_base_link: type fixed, parent world, child base_link
- joint panda_joint_base: parent world -> base_link
